Commit message: upload combined moveit2

File: main_description/urdf/m0609_rg2.urdf (robot description, URDF)
Before this commit: robot m0609, 17 links, 16 joints
Links:
- removed link base
- removed link tool0
Joints:
- removed joint base_link-base
- removed joint joint_6-tool0
- removed joint tool0-cylinder_link
- removed joint tool0-gripper_base_link
- added joint link6-cylinder_link: type fixed, parent link_6, child cylinder_link, origin xyz=0 0 0.005 rpy=0 -1.5707 0
- added joint link6-gripper_base_link: type fixed, parent cylinder_link, child gripper_base_link, origin xyz=0 0 0 rpy=0 0 0

Commit message: modify urdf and upload meshes

File: main_description/urdf/m0609_rg2.urdf (robot description, URDF)
Before this commit: robot m0609, 15 links, 14 joints
Links:
- link gripper_base_link: geometry collision mesh filename=package://main_description/meshes/collision/RG2_Hand_col.STL; visual mesh filename=package://main_description/meshes/visual/RG2_Hand_vis.STL
- link l_finger_link: geometry collision mesh filename=package://main_description/meshes/collision/RG2_LeftFinger_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; visual mesh filename=package://main_description/meshes/visual/RG2_LeftFinger_vis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
- link l_moment_arm_link: geometry collision mesh filename=package://main_description/meshes/collision/RG2_LeftMomentA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; visual mesh filename=package://main_description/meshes/visual/RG2_LeftMomentArm_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
- link l_truss_arm_link: geometry collision mesh filename=package://main_description/meshes/collision/RG2_LeftTrussAr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; visual mesh filename=package://main_description/meshes/visual/RG2_LeftTrussArm_v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
- link r_finger_link: geometry collision mesh filename=package://main_description/meshes/collision/RG2_RightFinger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; visual mesh filename=package://main_description/meshes/visual/RG2_RightFinger_vi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
- link r_moment_arm_link: geometry collision mesh filename=package://main_description/meshes/collision/RG2_RightMoment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; visual mesh filename=package://main_description/meshes/visual/RG2_RightMomentArm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
- link r_truss_arm_link: geometry collision mesh filename=package://main_description/meshes/collision/RG2_RightTrussA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; visual mesh filename=package://main_description/meshes/visual/RG2_RightTrussArm_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

Commit message: upload Unfinished code

File: main_description/urdf/m0609_rg2.urdf (robot description, URDF)
Before this commit: robot m0609, 15 links, 14 joints
Links:
- added link base
- added link camera_depth_optical_frame
Joints:
- added joint base_link-base: type fixed, parent base_link, child base, origin xyz=0 0 0.450 rpy=0 0 0
- added joint camera_to_tool: type fixed, parent cylinder_link, child camera_depth_optical_frame, origin xyz=0 0 0.0 rpy=0 -1.5707 0

File: rokey_moveit2/config/m0609.ros2_control.xacro (robot description, xacro)
@@ -2,5 +2,5 @@
 <robot xmlns:xacro="http://www.ros.org/wiki/xacro">
     <xacro:macro name="m0609_ros2_control" params="name initial_positions_file">
-        <xacro:property name="initial_positions" value="${load_yaml(initial_positions_file)['initial_positions']}"/>
+        <xacro:property name="initial_positions" value="${xacro.load_yaml(initial_positions_file)['initial_positions']}"/>
         <ros2_control name="${name}" type="system">
             <hardware>
